File: pcb/Flake.kicad_pcb (KiCad board)
At the start: 2 copper layers, 284 x 93.6 mm, 152 parts, among them J1 USB_C_Receptacle_PowerOnly_6P, J2 USB_C_Receptacle_PowerOnly_6P, SW1 SW_Push, SW10 SW_Push, SW11 SW_Push, SW12 SW_Push, SW13 SW_Push, SW14 SW_Push, SW15 SW_Push, SW16 SW_Push, SW17 SW_Push, SW18 SW_Push, SW19 SW_Push, SW2 SW_Push, SW20 SW_Push, SW21 SW_Push, SW22 SW_Push, SW23 SW_Push, SW24 SW_Push, SW25 SW_Push, SW26 SW_Push, SW27 SW_Push, SW28 SW_Push, SW29 SW_Push, SW3 SW_Push, SW30 SW_Push, SW31 SW_Push, SW32 SW_Push, SW33 SW_Push, SW34 SW_Push, SW35 SW_Push, SW36 SW_Push, SW37 SW_Push, SW38 SW_Push, SW39 SW_Push, SW4 SW_Push, SW40 SW_Push, SW41 SW_Push, SW42 SW_Push, SW43 SW_Push, SW44 SW_Push, SW45 SW_Push, SW46 SW_Push, SW5 SW_Push, SW6 SW_Push, SW7 SW_Push, SW8 SW_Push, SW9 SW_Push, U1 ProMicro, U2 ProMicro

Commit message: docs: add bill of materials
Parts:
- SW1, SW10, SW11, SW12, SW13, SW14, SW15, SW16, SW17, SW18, SW19, SW2, SW20, SW21, SW22, SW23, SW24, SW25, SW26, SW27, SW28, SW29, SW3, SW30, SW31, SW32, SW33, SW34, SW35, SW36, SW37, SW38, SW39, SW4, SW40, SW41, SW42, SW43, SW44, SW45, SW46, SW5, SW6, SW7, SW8, SW9: footprint axseem:SW_MX_Choch-v1v2_Hotswap -> axseem:SW_MX_Choc-v1v2_Hotswap
- moved RSW1 0.38 mm to (203.5, 136.2)
- moved RSW2 0.38 mm to (214.5, 136.2)
Connections:
- J1 pad S1: unconnected-(J1-SHIELD-PadS1)_1 -> LGND
- J2 pad S1: unconnected-(J2-SHIELD-PadS1)_2 -> RGND
Routing:
- net RGND: track 147.7 -> 161.6 mm
- net LGND: track 172.5 -> 185.2 mm
Other:
- outline, holes or cut-outs redrawn

Commit message: pcb: smd controller footprint
use smd prom-micro footprint
easier to break off the last column
wider controller cutout
ground usb shield
reroute some paths
minimse a chance of damaging the pcb after brakeing off the pinky column
edit silkscreen
Parts:
- added REF**: Hole_0.5mm, axseem:Hole_0.5mm, F.Cu at (86.2, 123.0)
- added REF**: Hole_0.5mm, axseem:Hole_0.5mm, F.Cu at (331.8, 123.0)
- added REF**: Hole_0.5mm, axseem:Hole_0.5mm, F.Cu at (331.8, 142.0)
- added REF**: Hole_0.5mm, axseem:Hole_0.5mm, F.Cu at (86.2, 142.0)
- added REF**: Hole_0.5mm, axseem:Hole_0.5mm, F.Cu at (86.2, 161.0)
- added REF**: Hole_0.5mm, axseem:Hole_0.5mm, F.Cu at (331.8, 161.0)
- U1, U2: footprint axseem:ProMicro -> axseem:ProMicro_SMD
- moved RSW1 0.12 mm to (203.6, 136.2)
- moved RSW2 0.12 mm to (214.4, 136.2)
Routing:
- net RData: track 8.19 -> 4.66 mm, vias 0 -> 2
- net LCol 1: track 180.2 -> 182.0 mm, vias 0 -> 1
- net LRow 0: track 129.9 -> 131.1 mm
- net RRow 0: track 160.0 -> 160.7 mm
- net LReset: track 31.6 -> 31.1 mm, vias 1 -> 2
- net RCol 0: track 169.4 -> 169.0 mm, vias 0 -> 1
- net LCol 0: track 179.2 -> 179.5 mm, vias 0 -> 1
- net LData: track 68.2 -> 68.4 mm, vias 0 -> 2
- net RVCC: track 66.3 -> 66.4 mm, vias 4 -> 5
- net RReset: track 47.3 -> 47.1 mm, vias 2 -> 4
- net RGND: vias 5 -> 8
- net RRaw: vias 4 -> 5
- net RCol 4: vias 0 -> 1
- net RCol 3: vias 0 -> 1
- net RCol 2: vias 0 -> 1
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Other:
- outline, holes or cut-outs redrawn
- board text added: "Anywhy Flake by @axseem v0.2.0"
- board text removed: "Anywhy Flake by @axseem v0.1.1"
