File: pcb/right.kicad_sch (KiCad schematic)
At the start: 56 parts, among them J2 USB_C_Receptacle_PowerOnly_6P, SW24 SW_Push, SW25 SW_Push, SW26 SW_Push, SW27 SW_Push, SW28 SW_Push, SW29 SW_Push, SW30 SW_Push, SW31 SW_Push, SW32 SW_Push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

Commit message: docs: add bill of materials
Connections:
- net RGND: now also J2.S1 (SHIELD)
- no-connect marks 8 -> 7
Changed lines of the file:
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@@
 	)
 	(no_connect
-		(at 93.98 58.42)
-	)
-	(no_connect
 		(at 29.21 46.99)
 	)
@@
 					(unit 1)
 				)
+			)
+		)
+	)
+	(symbol
+		(lib_id "power:GND")
+		(at 93.98 58.42 0)
+		(unit 1)
+		(exclude_from_sim no)
+		(in_bom yes)
+		(on_board yes)
+		(dnp no)
+		(property "Reference" "#PWR010"
+			(at 93.98 64.77 0)
+			(effects
+				(font
+					(size 1.27 1.27)
+				)
+				(hide yes)
+			)
+		)
+		(property "Value" "RGND"
+			(at 93.98 63.5 0)
+			(effects
+				(font
+					(size 1.27 1.27)
+				)
+			)
+		)
+		(property "Footprint" ""
+			(at 93.98 58.42 0)
+			(effects
+				(font
+					(size 1.27 1.27)
+				)
+				(hide yes)
+			)
+		)
+		(property "Datasheet" ""
+			(at 93.98 58.42 0)
+			(effects
+				(font
+					(size 1.27 1.27)
+				)
+				(hide yes)
+			)
+		)
+		(property "Description" "Power symbol creates a global label with name \"GND\" , ground"
+			(at 93.98 58.42 0)
+			(effects
+				(font
+					(size 1.27 1.27)
+				)
+				(hide yes)
+			)
+		)
+		(pin "1"
+		)
+		(instances
+			(project "Flake"
+				(path "/90c8b5ef-2115-4ce5-9f08-3facf16c5dc1/d5bac6f5-3ae0-4cc7-8f72-825f2fad23e6"
+					(reference "#PWR010")
+					(unit 1)
+				)

Commit message: pcb: smd controller footprint
use smd prom-micro footprint
easier to break off the last column
wider controller cutout
ground usb shield
reroute some paths
minimse a chance of damaging the pcb after brakeing off the pinky column
edit silkscreen
Parts:
- U2: footprint axseem:ProMicro -> axseem:ProMicro_SMD
Changed lines of the file:
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@@
 			)
 		)
-		(property "Footprint" "axseem:ProMicro"
+		(property "Footprint" "axseem:ProMicro_SMD"
 			(at 49.53 72.39 0)
 			(effects

Commit message: updates
Parts:
- removed BT2: Battery, axseem:JST_1.25mm_mid-mount, symbol Device:Battery
- removed D24, D30, D36, D42, D43, D44: D, axseem:D_SOD-123_Handsoldering, symbol Device:D
- removed H10, H7: MountingHole, MountingHole:MountingHole_2.2mm_M2, symbol Mechanical:MountingHole
- removed J2: USB_C_Receptacle_PowerOnly_6P, axseem:USB-C_6Pin_Mid-mount, symbol Connector:USB_C_Receptacle_PowerOnly_6P
- removed SW24, SW30, SW36, SW42, SW43, SW44: SW_Push, axseem:SW_MX_Choc-v1v2_Hotswap, symbol Switch:SW_Push
- removed U2: ProMicro, axseem:ProMicro_SMD, symbol kbd:ProMicro
- added R_BATT1: Conn_01x02, Connector_JST:JST_PH_S2B-PH-K_1x02_P2.00mm_Horizontal, symbol Connector_Generic:Conn_01x02
- added R_DISPLAY1: nice!view, axseem:nice_view, symbol nice_nano:nice!view
- added R_MCU1: nice_nano, axseem:nice_nano, symbol nice_nano:nice_nano
- added R_POWER_SW1: SW_SPDT, axseem:smt-slider-switch, symbol Switch:SW_SPDT
- R_RSW1: renamed from RSW2; footprint axseem:TS-1289VE-4 -> axseem:SMD_RESET
Connections:
- net RCol 5 is gone; now on net RCol 4: SW29.1, SW35.1, SW41.1, SW46.1
- net RCol 0: now also SW25.1, SW31.1, SW37.1, R_MCU1.17 (P1.15)
- net RCol 1: now also SW26.1, SW32.1, SW38.1, R_MCU1.16 (P1.13); no longer SW25.1, SW31.1, SW37.1
- net RCol 2: now also SW27.1, SW33.1, SW39.1, R_MCU1.15 (P1.11); no longer SW26.1, SW32.1, SW38.1
- net RCol 3: now also SW28.1, SW34.1, SW40.1, SW45.1, R_MCU1.14 (NFC2/P0.10); no longer SW27.1, SW33.1, SW39.1
- net RCol 4: now also R_MCU1.13 (NFC1/P0.09); no longer SW28.1, SW34.1, SW40.1, SW45.1
- net RGND: now also R_BATT1.1 (Pin_1), R_DISPLAY1.4 (GND), R_MCU1.23 (GND), R_MCU1.3 (GND), R_MCU1.4 (GND)
- net RRaw: now also R_MCU1.24 (BATIN/P0.04), R_POWER_SW1.3 (C)
- net RReset: now also R_MCU1.22 (RST)
- net RRow 0: now also R_MCU1.9 (P1.00)
- net RRow 1: now also R_MCU1.10 (P0.11)
- net RRow 2: now also R_MCU1.11 (P1.04)
- net RRow 3: now also R_MCU1.12 (P1.06)
- new net +3.3V: R_DISPLAY1.3 (VCC), R_MCU1.21 (VCC)
- new net R_BT+: R_BATT1.2 (Pin_2), R_POWER_SW1.2 (B)
- new net R_MOSI: R_DISPLAY1.1 (MOSI), R_MCU1.5 (P0.17)
- new net R_NVCS: R_DISPLAY1.5 (CS), R_MCU1.1 (TX0/P0.06)
- new net R_SCK: R_DISPLAY1.2 (SCK), R_MCU1.6 (P0.20)
- no-connect marks 7 -> 10
Other:
- note added: "Nice!NanoV2"
- note added: "Nice!View"
- note removed: "ProMicro module"
- note removed: "USB port"
- moved on the sheet: R_RSW1

Commit message: update
Connections:
- net +3.3V renamed R_VCC
Changed lines of the file:
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@@
 	(wire
 		(pts
-			(xy 92.71 64.77) (xy 97.79 64.77)
-		)
-		(stroke
-			(width 0)
-			(type default)
-		)
-	)
-	(wire
-		(pts
 			(xy 29.21 107.95) (xy 55.88 107.95)
 		)
@@
 	(wire
 		(pts
-			(xy 68.58 33.02) (xy 81.28 33.02)
-		)
-		(stroke
-			(width 0)
-			(type default)
-		)
-	)
-	(wire
-		(pts
-			(xy 97.79 64.77) (xy 97.79 48.26)
-		)
-		(stroke
-			(width 0)
-			(type default)
-		)
-	)
-	(wire
-		(pts
 			(xy 73.66 100.33) (xy 73.66 113.03)
 		)
@@
 		)
 	)
+	(global_label "R_VCC"
+		(shape input)
+		(at 68.58 33.02 0)
+		(fields_autoplaced yes)
+		(effects
+			(font
+				(size 1.27 1.27)
+			)
+			(justify left)
+		)
+		(property "Intersheetrefs" "${INTERSHEET_REFS}"
+			(at 77.4314 33.02 0)
+			(effects
+				(font
+					(size 1.27 1.27)
+				)
+				(justify left)
+				(hide yes)
+			)
+		)
+	)
 	(global_label "RReset"
 		(shape input)
@@
 	)
 	(global_label "R_SCK"
-		(shape output)
+		(shape input)
 		(at 33.02 38.1 180)
 		(fields_autoplaced yes)
@@
 		)
 	)
+	(global_label "R_VCC"
+		(shape input)
+		(at 97.79 48.26 270)
+		(fields_autoplaced yes)
+		(effects
+			(font
+				(size 1.27 1.27)
+			)
+			(justify right)
+		)
+		(property "Intersheetrefs" "${INTERSHEET_REFS}"
+			(at 97.79 57.1114 90)
+			(effects
+				(font
+					(size 1.27 1.27)
+				)
+				(justify right)
+				(hide yes)
+			)
+		)
+	)
 	(global_label "R_MOSI"
 		(shape input)
@@
 	)
 	(global_label "R_NVCS"
-		(shape output)
+		(shape input)
 		(at 33.02 25.4 180)
 		(fields_autoplaced yes)
@@
 	)
 	(global_label "R_MOSI"
-		(shape output)
+		(shape input)
 		(at 33.02 35.56 180)
 		(fields_autoplaced yes)
@@
 	)
 	(symbol
-		(lib_id "power:+3.3V")
-		(at 81.28 33.02 180)
-		(unit 1)
-		(exclude_from_sim no)
-		(in_bom yes)
-		(on_board yes)
-		(dnp no)
-		(property "Reference" "#PWR07"
-			(at 81.28 29.21 0)
-			(effects
-				(font
-					(size 1.27 1.27)
-				)
-				(hide yes)
-			)
-		)
-		(property "Value" "+3.3V"
-			(at 81.28 37.338 0)
-			(effects
-				(font
-					(size 1.27 1.27)
-				)
-			)
-		)
-		(property "Footprint" ""
-			(at 81.28 33.02 0)
-			(effects
-				(font
-					(size 1.27 1.27)
-				)
-				(hide yes)
-			)
-		)
-		(property "Datasheet" ""
-			(at 81.28 33.02 0)
-			(effects
-				(font
-					(size 1.27 1.27)
-				)
-				(hide yes)
-			)
-		)
-		(property "Description" "Power symbol creates a global label with name \"+3.3V\""
-			(at 81.28 33.02 0)
-			(effects
-				(font
-					(size 1.27 1.27)
-				)
-				(hide yes)
-			)
-		)
-		(pin "1"
-		)
-		(instances
-			(project "Flake"
-				(path "/90c8b5ef-2115-4ce5-9f08-3facf16c5dc1/d5bac6f5-3ae0-4cc7-8f72-825f2fad23e6"
-					(reference "#PWR07")
-					(unit 1)
-				)
-			)
-		)
-	)
-	(symbol
 		(lib_id "Device:D")
 		(at 83.82 116.84 90)
@@
 					(unit 1)
 				)
-			)
-		)
-	)
-	(symbol
-		(lib_id "power:+3.3V")
-		(at 92.71 64.77 0)
-		(unit 1)
-		(exclude_from_sim no)
-		(in_bom yes)
-		(on_board yes)
-		(dnp no)
-		(property "Reference" "#PWR08"
-			(at 92.71 68.58 0)
-			(effects
-				(font
-					(size 1.27 1.27)
-				)
-				(hide yes)
-			)
-		)
-		(property "Value" "+3.3V"
-			(at 92.71 60.452 0)
-			(effects
-				(font
-					(size 1.27 1.27)
-				)
-			)
-		)
-		(property "Footprint" ""
-			(at 92.71 64.77 0)
-			(effects
-				(font
-					(size 1.27 1.27)
-				)
-				(hide yes)
-			)
-		)
-		(property "Datasheet" ""
-			(at 92.71 64.77 0)
-			(effects
-				(font
-					(size 1.27 1.27)
-				)
-				(hide yes)
-			)
-		)
-		(property "Description" "Power symbol creates a global label with name \"+3.3V\""
-			(at 92.71 64.77 0)
-			(effects
-				(font
-					(size 1.27 1.27)
-				)
-				(hide yes)
-			)
-		)
-		(pin "1"
-		)
-		(instances
-			(project "Flake"
-				(path "/90c8b5ef-2115-4ce5-9f08-3facf16c5dc1/d5bac6f5-3ae0-4cc7-8f72-825f2fad23e6"
-					(reference "#PWR08")
-					(unit 1)
-				)
